File: kicad-project/powerpack.sch (KiCad schematic (older format))
At the start: 8 parts, among them J1 Power_in 3.3-15V, J2.1 Vout +3.3V, J2.2 Vout GND, J3.1 Vin 3.3V-15V, J3.2 Vin GND, U1 MCP1703T-3302E_CB

Commit message: Update
Parts:
- added J4: ADC, TestPoint:TestPoint_Pad_2.5x2.5mm, symbol Connector:Conn_01x01_Male
- added R1, R2: R, Resistor_SMD:R_1206_3216Metric_Pad1.30x1.75mm_HandSolder, symbol Device:R
Connections:
- net GND: now also R2.2
- net VCC: now also R1.1
- new net: J4.1 (Pin_1), R1.2, R2.1
Changed lines of the file:
@@
 Wire Wire Line
 	3900 1750 3900 2000
+$Comp
+L Device:R R1
+U 1 1 60AE73CA
+P 1600 2400
+F 0 "R1" H 1670 2446 50  0000 L CNN
+F 1 "R" H 1670 2355 50  0000 L CNN
+F 2 "Resistor_SMD:R_1206_3216Metric_Pad1.30x1.75mm_HandSolder" V 1530 2400 50  0001 C CNN
+F 3 "~" H 1600 2400 50  0001 C CNN
+	1    1600 2400
+	1    0    0    -1
+$EndComp
+$Comp
+L Device:R R2
+U 1 1 60AE7AA8
+P 1600 2850
+F 0 "R2" H 1670 2896 50  0000 L CNN
+F 1 "R" H 1670 2805 50  0000 L CNN
+F 2 "Resistor_SMD:R_1206_3216Metric_Pad1.30x1.75mm_HandSolder" V 1530 2850 50  0001 C CNN
+F 3 "~" H 1600 2850 50  0001 C CNN
+	1    1600 2850
+	1    0    0    -1
+$EndComp
+$Comp
+L power:GND #PWR0102
+U 1 1 60AE8111
+P 1600 3050
+F 0 "#PWR0102" H 1600 2800 50  0001 C CNN
+F 1 "GND" H 1605 2877 50  0000 C CNN
+F 2 "" H 1600 3050 50  0001 C CNN
+F 3 "" H 1600 3050 50  0001 C CNN
+	1    1600 3050
+	1    0    0    -1
+$EndComp
+Wire Wire Line
+	1600 3000 1600 3050
+Wire Wire Line
+	1600 2700 1600 2600
+Wire Wire Line
+	1600 2250 1600 2100
+Connection ~ 1600 2100
+$Comp
+L Connector:Conn_01x01_Male J4
+U 1 1 60AE930E
+P 1300 2600
+F 0 "J4" H 1408 2781 50  0000 C CNN
+F 1 "ADC" H 1408 2690 50  0000 C CNN
+F 2 "TestPoint:TestPoint_Pad_2.5x2.5mm" H 1300 2600 50  0001 C CNN
+F 3 "~" H 1300 2600 50  0001 C CNN
+	1    1300 2600
+	1    0    0    -1
+$EndComp
+Wire Wire Line
+	1500 2600 1600 2600
+Connection ~ 1600 2600
+Wire Wire Line
+	1600 2600 1600 2550
 $EndSCHEMATC
